Commit message: lowered mu values. need to play with correct balance that allows for motion while limiting spawn drift

File: src/MRP_Description/urdf/MRP_Gazebo_Properties.xacro (robot description, xacro)
@@ -2,6 +2,6 @@
 <robot xmlns:xacro="http://www.ros.org/wiki/xacro">
     <!--                PROPERTIES                 -->
-    <xacro:property name = 'mu1' value = '10'/>
-    <xacro:property name = 'mu2' value = '10'/>
+    <xacro:property name = 'mu1' value = '0.2'/>
+    <xacro:property name = 'mu2' value = '0.2'/>
     <!--                STRUCTURAL LINKS                 -->
     <gazebo reference = 'chassis_link'>

Commit message: reduced the mu values to something more reasonable

File: src/MRP_Description/urdf/MRP_Gazebo_Properties.xacro (robot description, xacro)
@@ -2,6 +2,6 @@
 <robot xmlns:xacro="http://www.ros.org/wiki/xacro">
     <!--                PROPERTIES                 -->
-    <xacro:property name = 'mu1' value = '0.2'/>
-    <xacro:property name = 'mu2' value = '0.2'/>
+    <xacro:property name = 'mu1' value = '1'/>
+    <xacro:property name = 'mu2' value = '1'/>
     <!--                STRUCTURAL LINKS                 -->
     <gazebo reference = 'chassis_link'>
