Commit message: tweaked URDF for use in Gazebo

File: src/MRP_Description/urdf/MRP.urdf.xacro (robot description, xacro)
@@ -4,5 +4,4 @@
     <xacro:include filename="MRP_Body.xacro"/>
     <xacro:include filename="MRP_Gazebo_Properties.xacro"/>
-    <!-- <xacro:include filename="MRP_Peripherals.xacro"/> -->
-    <!-- could also include the gazebo properties here -->
+    <xacro:include filename="MRP_Gazebo_Control.xacro"/>
 </robot>

File: src/MRP_Description/urdf/MRP_Body.xacro (robot description, xacro)
@@ -2,5 +2,6 @@
 <!-- start the robot tag here -->
 <robot xmlns:xacro="http://www.ros.org/wiki/xacro">
-    <!--                MATERIALS:                 -->
+    <!--                PROPERTIES:                 -->
+    <xacro:property name='a' value='4'/>
     <material name = "black">
         <color rgba = "0.1 0.1 0.1 1"/>
@@ -17,6 +18,7 @@
         <parent link = 'base_link'/>
         <child link = 'chassis_link'/>
-        <origin xyz = "0 0 0.122"/>
-    </joint>
+        <origin xyz = "0 0 0.125"/>
+    </joint>
+    <!-- 0.122 -->
     <!-- rear left motor to chassis joint -->
     <joint name = 'C_RLM_joint' type = 'fixed'>
@@ -100,5 +102,11 @@
         <inertial>
             <mass value = '0.27224'/>
-            <inertia ixx = '2.853307738e-3' ixy = '0' ixz = '0' iyy = '1.442962747e-3' iyz = '0' izz = '4.291733152e-3'/>
+            <inertia
+                        ixx = '${a * 2.853307738e-3}'
+                        ixy = '${a * 1e-6}'
+                        ixz = '${a * 1e-6}'
+                        iyy = '${a* 1.442962747e-3}'
+                        iyz = '${a * 1e-6}'
+                        izz = '${a * 4.291733152e-3}'/>
         </inertial>
     </link>
@@ -120,5 +128,11 @@
         <inertial>
             <mass value = '0.08492'/>
-            <inertia ixx = '3.682697333e-5' ixy = '0' ixz = '0' iyy = '4.670883067e-4' iyz = '0' izz = '4.685319467e-4'/>
+            <inertia
+                        ixx = '${a * 3.682697333e-5}'
+                        ixy = '${a * 1e-6}'
+                        ixz = '${a * 1e-6}'
+                        iyy = '${a * 4.670883067e-4}'
+                        iyz = '${a * 1e-6}'
+                        izz = '${a * 4.685319467e-4}'/>
         </inertial>
     </link>
@@ -141,5 +155,11 @@
         <inertial>
             <mass value = '0.1579'/>
-            <inertia ixx = '5.188001875e-5' ixy = '0' ixz = '0' iyy = '5.188001875e-5' iyz = '0' izz = '2.70206375e-5'/>
+            <inertia
+                        ixx = '${a * 5.188001875e-5}'
+                        ixy = '${a * 1e-6}'
+                        ixz = '${a * 1e-6}'
+                        iyy = '${a * 5.188001875e-5}'
+                        iyz = '${a * 1e-6}'
+                        izz = '${a * 2.70206375e-5}'/>
         </inertial>
     </link>
@@ -161,5 +181,11 @@
         <inertial>
             <mass value = '0.1579'/>
-            <inertia ixx = '5.188001875e-5' ixy = '0' ixz = '0' iyy = '5.188001875e-5' iyz = '0' izz = '2.70206375e-5'/>
+            <inertia
+                        ixx = '${a * 5.188001875e-5}'
+                        ixy = '${a * 1e-6}'
+                        ixz = '${a * 1e-6}'
+                        iyy = '${a * 5.188001875e-5}'
+                        iyz = '${a * 1e-6}'
+                        izz = '${a * 2.70206375e-5}'/>
         </inertial>
     </link>
@@ -181,5 +207,11 @@
         <inertial>
             <mass value = '0.1579'/>
-            <inertia ixx = '5.188001875e-5' ixy = '0' ixz = '0' iyy = '5.188001875e-5' iyz = '0' izz = '2.70206375e-5'/>
+            <inertia
+                        ixx = '${a * 5.188001875e-5}'
+                        ixy = '${a * 1e-6}'
+                        ixz = '${a * 1e-6}'
+                        iyy = '${a * 5.188001875e-5}'
+                        iyz = '${a * 1e-6}'
+                        izz = '${a * 2.70206375e-5}'/>
         </inertial>
     </link>
@@ -201,5 +233,11 @@
         <inertial>
             <mass value = '0.1579'/>
-            <inertia ixx = '5.188001875e-5' ixy = '0' ixz = '0' iyy = '5.188001875e-5' iyz = '0' izz = '2.70206375e-5'/>
+            <inertia
+                        ixx = '${a * 5.188001875e-5}'
+                        ixy = '${a * 1e-6}'
+                        ixz = '${a * 1e-6}'
+                        iyy = '${a * 5.188001875e-5}'
+                        iyz = '${a * 1e-6}'
+                        izz = '${a * 2.70206375e-5}'/>
         </inertial>
     </link>
@@ -222,5 +260,11 @@
         <inertial>
             <mass value = "0.147595"/>
-            <inertia ixx="3.20634763e-4" ixy="0" ixz="0" iyy="3.20634763e-4" iyz="0" izz="6.314298594e-4"/>
+            <inertia
+                        ixx = "${a * 3.20634763e-4}"
+                        ixy = "${a * 1e-6}"
+                        ixz = "${a * 1e-6}"
+                        iyy = "${a * 3.20634763e-4}"
+                        iyz = "${a * 1e-6}"
+                        izz = "${a * 6.314298594e-4}"/>
         </inertial>
     </link>
@@ -242,5 +286,11 @@
         <inertial>
             <mass value = "0.147595"/>
-            <inertia ixx="3.20634763e-4" ixy="0" ixz="0" iyy="3.20634763e-4" iyz="0" izz="6.314298594e-4"/>
+            <inertia
+                        ixx = "${a * 3.20634763e-4}"
+                        ixy = "${a * 1e-6}"
+                        ixz = "${a * 1e-6}"
+                        iyy = "${a * 3.20634763e-4}"
+                        iyz = "${a * 1e-6}"
+                        izz = "${a * 6.314298594e-4}"/>
         </inertial>
     </link>
@@ -262,5 +312,11 @@
         <inertial>
             <mass value = "0.147595"/>
-            <inertia ixx="3.20634763e-4" ixy="0" ixz="0" iyy="3.20634763e-4" iyz="0" izz="6.314298594e-4"/>
+            <inertia
+                        ixx = "${a * 3.20634763e-4}"
+                        ixy = "${a * 1e-6}"
+                        ixz = "${a * 1e-6}"
+                        iyy = "${a * 3.20634763e-4}"
+                        iyz = "${a * 1e-6}"
+                        izz = "${a * 6.314298594e-4}"/>
         </inertial>
     </link>
@@ -282,5 +338,11 @@
         <inertial>
             <mass value = "0.147595"/>
-            <inertia ixx="3.20634763e-4" ixy="0" ixz="0" iyy="3.20634763e-4" iyz="0" izz="6.314298594e-4"/>
+            <inertia
+                        ixx = "${a * 3.20634763e-4}"
+                        ixy = "${a * 1e-6}"
+                        ixz = "${a * 1e-6}"
+                        iyy = "${a * 3.20634763e-4}"
+                        iyz = "${a * 1e-6}"
+                        izz = "${a * 6.314298594e-4}"/>
         </inertial>
     </link>

File: src/MRP_Description/urdf/MRP_Gazebo_Properties.xacro (robot description, xacro)
@@ -1,4 +1,7 @@
 <?xml version="1.0"?>
 <robot xmlns:xacro="http://www.ros.org/wiki/xacro">
+    <!--                PROPERTIES:                 -->
+    <xacro:property name = 'mu1' value = '1.0'/>
+    <xacro:property name = 'mu2' value = '1.0'/>
     <!--                STRUCTURAL LINKS:                 -->
     <gazebo reference = 'chassis_link'>
@@ -24,21 +27,21 @@
     <gazebo reference = 'rear_left_wheel'>
         <material>Gazebo/Grey</material>
-        <mu1 value="0.8" />
-        <mu2 value="0.6" />
+        <mu1 value="${mu1}" />
+        <mu2 value="${mu2}" />
     </gazebo>
     <gazebo reference = 'rear_right_wheel'>
         <material>Gazebo/Grey</material>
-        <mu1 value="0.8" />
-        <mu2 value="0.6" />
+        <mu1 value="${mu1}" />
+        <mu2 value="${mu2}" />
     </gazebo>
     <gazebo reference = 'front_left_wheel'>
         <material>Gazebo/Grey</material>
-        <mu1 value="0.8" />
-        <mu2 value="0.6" />
+        <mu1 value="${mu1}" />
+        <mu2 value="${mu2}" />
     </gazebo>
     <gazebo reference = 'front_right_wheel'>
         <material>Gazebo/Grey</material>
-        <mu1 value="0.8" />
-        <mu2 value="0.6" />
+        <mu1 value="${mu1}" />
+        <mu2 value="${mu2}" />
     </gazebo>
 </robot>
