Commit message: various URDF changes

File: src/MRP_Description/urdf/MRP.urdf.xacro (robot description, xacro)
@@ -1,7 +1,15 @@
 <?xml version="1.0"?>
-<robot name='MRP.urdf' xmlns:xacro="http://www.ros.org/wiki/xacro">
+<robot name='MRP' xmlns:xacro="http://www.ros.org/wiki/xacro">
+    <xacro:arg name='use_ros2_control' default='true'/>
     <!-- include the xacro files that contain our robot -->
-    <xacro:include filename="MRP_Body.xacro"/>
-    <xacro:include filename="MRP_Gazebo_Properties.xacro"/>
-    <xacro:include filename="MRP_Gazebo_Control.xacro"/>
+    <xacro:include filename = "MRP_Body.xacro"/>
+    <xacro:include filename = "MRP_Gazebo_Properties.xacro"/>
+    <!-- if we want to use ros2 control: -->
+    <xacro:if value ="$(arg use_ros2_control)">
+        <xacro:include filename = "MRP_Control.xacro"/>
+    </xacro:if>
+    <!-- if we want to use gazebo control: -->
+    <xacro:unless value = "$(arg use_ros2_control)">
+        <xacro:include filename = "MRP_Gazebo_Control.xacro"/>
+    </xacro:unless>
 </robot>

File: src/MRP_Description/urdf/MRP_Body.xacro (robot description, xacro)
@@ -1,246 +1,60 @@
 <?xml version="1.0"?>
-<!-- start the robot tag here -->
 <robot xmlns:xacro="http://www.ros.org/wiki/xacro">
     <!--                PROPERTIES:                 -->
-    <xacro:property name='a' value='6'/>
+    <xacro:property name = 'a' value = '1'/>
+    <xacro:property name = 'b' value = '4'/>
+    <xacro:property name = 'd' value = '0.2'/>
     <material name = "black">
         <color rgba = "0.1 0.1 0.1 1"/>
-    </material>
-    <material name = "grey">
-        <color rgba = "0.5 0.5 0.5 1"/>
     </material>
     <material name = "red">
         <color rgba = "1 0 0 1"/>
     </material>
-    <!--                JOINTS:                 -->
-    <!-- chassis to base link joint -->
-    <joint name = 'B_C_joint' type = 'fixed'>
-        <parent link = 'base_link'/>
-        <child link = 'chassis_link'/>
-        <origin xyz = "0 0 0.125"/>
-    </joint>
-    <!-- 0.122 -->
-    <!-- rear left motor to chassis joint -->
-    <joint name = 'C_RLM_joint' type = 'fixed'>
-        <parent link = 'chassis_link'/>
-        <child link = 'rear_left_motor'/>
-        <origin xyz = '-0.1355 0.1015 -0.003' rpy = '-1.570796 0 0'/>
-    </joint>
-    <!-- rear left wheel to rear left motor joint -->
-    <joint name = 'RLM_RLW_joint' type = 'continuous'>
-        <parent link = 'rear_left_motor'/>
-        <child link = 'rear_left_wheel'/>
-        <origin xyz = '0 0.0255 0.0425' rpy = '0 0 0'/>
-        <axis xyz = '0 0 1'/>
-    </joint>
-    <!-- rear right wheel to rear right motor joint -->
-    <joint name = 'RRM_RRW_joint' type = 'continuous'>
-        <parent link = 'rear_right_motor'/>
-        <child link = 'rear_right_wheel'/>
-        <origin xyz = '0 -0.0255 0.0425' rpy = '0 0 0'/>
-        <axis xyz = '0 0 -1'/>
-    </joint>
-    <!-- rear right motor to chassis joint -->
-    <joint name = 'C_RRM_joint' type = 'fixed'>
-        <parent link = 'chassis_link'/>
-        <child link = 'rear_right_motor'/>
-        <origin xyz = '-0.1355 -0.1015 -0.003' rpy = '1.570796 0 0'/>
-    </joint>
-    <!-- chassis to pendulum bracket joint -->
-    <joint name = 'C_to_PB_joint' type = 'revolute'>
-        <parent link = 'chassis_link'/>
-        <child link = 'pendulum_bracket_link'/>
-        <origin xyz = '0.1755 0 -0.010562'/>
-        <axis xyz = '1 0 0'/>
-        <limit lower = '-0.261799' upper ='0.261799' effort = '10' velocity = '1'/>
-    </joint>
-    <!-- front left motor to pendulum bracket joint -->
-    <joint name = 'PB_FLM_joint' type = 'fixed'>
-        <parent link = 'pendulum_bracket_link'/>
-        <child link = 'front_left_motor'/>
-        <origin xyz = '0 0.1015 -0.029438' rpy = '-1.570796 0 0'/>
-    </joint>
-    <!-- front left wheel to front left motor joint -->
-    <joint name = 'FLM_FLW_joint' type = 'continuous'>
-        <parent link = 'front_left_motor'/>
-        <child link = 'front_left_wheel'/>
-        <origin xyz = '0 -0.0115 0.0425' rpy = '0 0 0'/>
-        <axis xyz = '0 0 1'/>
-    </joint>
-    <!-- front right motor to pendulum bracket joint -->
-    <joint name = 'PB_FRM_joint' type = 'fixed'>
-        <parent link = 'pendulum_bracket_link'/>
-        <child link = 'front_right_motor'/>
-        <origin xyz = '0 -0.1015 -0.029438' rpy = '1.570796 0 0'/>
-    </joint>
-    <!-- front right wheel to front right motor joint -->
-    <joint name = 'FRM_FRW_joint' type = 'continuous'>
-        <parent link = 'front_right_motor'/>
-        <child link = 'front_right_wheel'/>
-        <origin xyz = '0 0.0115 0.0425' rpy = '0 0 0'/>
-        <axis xyz = '0 0 -1'/>
-    </joint>
-    <!--                STRUCTURAL LINKS:                 -->
+    <material name = "purple">
+        <color rgba = "0.25 0.15 0.25 1"/>
+    </material>
     <!-- base link -->
     <link name = "base_link">
     </link>
+    <!-- chassis to base link joint -->
+    <joint name = 'base_link_to_chassis_joint' type = 'fixed'>
+        <parent link = 'base_link'/>
+        <child link = 'chassis_link'/>
+        <origin xyz = '0 0 0.121'/>
+    </joint>
     <!-- chassis link -->
     <link name = 'chassis_link'>
         <visual>
-            <origin xyz = "0 0 0" rpy = "1.570796 0 0"/>
+            <origin xyz = '0 0 0' rpy = '1.570796 0 0'/>
             <geometry>
-                <mesh filename = "file://$(find MRP_Description)/meshes/chassis.stl" scale = "0.001 0.001 0.001"/>
+                <mesh filename = "file://$(find MRP_Description)/meshes/entire_chassis.stl" scale = "0.001 0.001 0.001"/>
             </geometry>
             <material name = 'black'/>
         </visual>
         <collision>
-            <origin xyz = "0 0 0" rpy = "1.570796 0 0"/>
+            <origin xyz = '0.02125 0 -0.02' rpy = '1.570796 0 0'/>
             <geometry>
-                <mesh filename = "file://$(find MRP_Description)/meshes/chassis.stl" scale = "0.001 0.001 0.001"/>
+                <box size = '0.3605 0.06 0.288'/>
             </geometry>
         </collision>
         <inertial>
-            <mass value = '0.27224'/>
+            <mass value = '1.0'/>
             <inertia
-                        ixx = '${a * 2.853307738e-3}'
-                        ixy = '${a * 1e-6}'
-                        ixz = '${a * 1e-6}'
-                        iyy = '${a* 1.442962747e-3}'
-                        iyz = '${a * 1e-6}'
-                        izz = '${a * 4.291733152e-3}'/>
+                ixx = '${a * 8.617577e-3}'
+                ixy = '${a * 9.10052e-4}'
+                ixz = '${a * 1e-8}'
+                iyy = '${a * 0.030175621}'
+                iyz = '${a * 1e-8}'
+                izz = '${a * 0.022585289}'/>
         </inertial>
     </link>
-    <!-- pendulum bracket link -->
-    <link name = 'pendulum_bracket_link'>
-        <visual>
-            <origin xyz = "0 0 -0.039438" rpy = "1.570796 0 0"/>
-            <geometry>
-                <mesh filename = "file://$(find MRP_Description)/meshes/pendulum_bracket.stl" scale = "0.001 0.001 0.001"/>
-            </geometry>
-            <material name = 'black'/>
-        </visual>
-        <collision>
-            <origin xyz = "0 0 -0.039438" rpy = "1.570796 0 0"/>
-            <geometry>
-                <mesh filename = "file://$(find MRP_Description)/meshes/pendulum_bracket.stl" scale = "0.001 0.001 0.001"/>
-            </geometry>
-        </collision>
-        <inertial>
-            <mass value = '0.08492'/>
-            <inertia
-                        ixx = '${a * 3.682697333e-5}'
-                        ixy = '${a * 1e-6}'
-                        ixz = '${a * 1e-6}'
-                        iyy = '${a * 4.670883067e-4}'
-                        iyz = '${a * 1e-6}'
-                        izz = '${a * 4.685319467e-4}'/>
-        </inertial>
-    </link>
-    <!--                MOTORS:                 -->
-    <!-- rear left motor link -->
-    <link name = 'rear_left_motor'>
-        <visual>
-            <origin xyz = "0 0.0185 0 " rpy = "0 0 3.141592"/>
-            <geometry>
-                <mesh filename = "file://$(find MRP_Description)/meshes/520_dc_gear_motor.stl" scale = "0.001 0.001 0.001"/>
-            </geometry>
-            <material name = 'red'/>
-        </visual>
-        <collision>
-            <origin xyz = "0 0.0185 0" rpy = "0 0 3.141592"/>
-            <geometry>
-                <mesh filename = "file://$(find MRP_Description)/meshes/520_dc_gear_motor.stl" scale = "0.001 0.001 0.001"/>
-            </geometry>
-        </collision>
-        <inertial>
-            <mass value = '0.1579'/>
-            <inertia
-                        ixx = '${a * 5.188001875e-5}'
-                        ixy = '${a * 1e-6}'
-                        ixz = '${a * 1e-6}'
-                        iyy = '${a * 5.188001875e-5}'
-                        iyz = '${a * 1e-6}'
-                        izz = '${a * 2.70206375e-5}'/>
-        </inertial>
-    </link>
-    <!-- rear right motor link -->
-    <link name = 'rear_right_motor'>
-        <visual>
-            <origin xyz = "0 -0.0185 0" rpy = "0 0 0"/>
-            <geometry>
-                <mesh filename = "file://$(find MRP_Description)/meshes/520_dc_gear_motor.stl" scale = "0.001 0.001 0.001"/>
-            </geometry>
-            <material name = 'red'/>
-        </visual>
-        <collision>
-            <origin xyz = "0 -0.0185 0" rpy = "0 0 0"/>
-            <geometry>
-                <mesh filename = "file://$(find MRP_Description)/meshes/520_dc_gear_motor.stl" scale = "0.001 0.001 0.001"/>
-            </geometry>
-        </collision>
-        <inertial>
-            <mass value = '0.1579'/>
-            <inertia
-                        ixx = '${a * 5.188001875e-5}'
-                        ixy = '${a * 1e-6}'
-                        ixz = '${a * 1e-6}'
-                        iyy = '${a * 5.188001875e-5}'
-                        iyz = '${a * 1e-6}'
-                        izz = '${a * 2.70206375e-5}'/>
-        </inertial>
-    </link>
-    <!-- front left motor -->
-    <link name = 'front_left_motor'>
-        <visual>
-            <origin xyz = "0 -0.0185 0" rpy = "0 0 3.141592"/>
-            <geometry>
-                <mesh filename = "file://$(find MRP_Description)/meshes/520_dc_gear_motor.stl" scale = "0.001 0.001 0.001"/>
-            </geometry>
-            <material name = 'red'/>
-        </visual>
-        <collision>
-            <origin xyz = "0 -0.0185 0" rpy = "0 0 3.141592"/>
-            <geometry>
-                <mesh filename = "file://$(find MRP_Description)/meshes/520_dc_gear_motor.stl" scale = "0.001 0.001 0.001"/>
-            </geometry>
-        </collision>
-        <inertial>
-            <mass value = '0.1579'/>
-            <inertia
-                        ixx = '${a * 5.188001875e-5}'
-                        ixy = '${a * 1e-6}'
-                        ixz = '${a * 1e-6}'
-                        iyy = '${a * 5.188001875e-5}'
-                        iyz = '${a * 1e-6}'
-                        izz = '${a * 2.70206375e-5}'/>
-        </inertial>
-    </link>
-    <!-- front right motor -->
-    <link name = 'front_right_motor'>
-        <visual>
-            <origin xyz = "0 0.0185 0" rpy = "0 0 0"/>
-            <geometry>
-                <mesh filename = "file://$(find MRP_Description)/meshes/520_dc_gear_motor.stl" scale = "0.001 0.001 0.001"/>
-            </geometry>
-            <material name = 'red'/>
-        </visual>
-        <collision>
-            <origin xyz = "0 0.0185 0" rpy = "0 0 0"/>
-            <geometry>
-                <mesh filename = "file://$(find MRP_Description)/meshes/520_dc_gear_motor.stl" scale = "0.001 0.001 0.001"/>
-            </geometry>
-        </collision>
-        <inertial>
-            <mass value = '0.1579'/>
-            <inertia
-                        ixx = '${a * 5.188001875e-5}'
-                        ixy = '${a * 1e-6}'
-                        ixz = '${a * 1e-6}'
-                        iyy = '${a * 5.188001875e-5}'
-                        iyz = '${a * 1e-6}'
-                        izz = '${a * 2.70206375e-5}'/>
-        </inertial>
-    </link>
-    <!--                WHEELS:                 -->
+    <!-- rear left wheel to chassis joint -->
+    <joint name = 'rear_left_wheel_joint' type = 'continuous'>
+        <parent link = 'chassis_link'/>
+        <child link = 'rear_left_wheel'/>
+        <origin xyz = '-0.1355 0.144 -0.0285' rpy = '-1.570796 0 0'/>
+        <axis xyz = '0 0 1'/>
+        <dynamics damping = '${d}' />
+    </joint>
     <!-- rear left wheel -->
     <link name = 'rear_left_wheel'>
@@ -250,23 +64,31 @@
                 <mesh filename = "file://$(find MRP_Description)/meshes/wheel_coupler_assembly.stl" scale = "0.001 0.001 0.001"/>
             </geometry>
-            <material name = 'grey'/>
+            <material name = 'purple'/>
         </visual>
         <collision>
-            <origin xyz = "0 0 0.012" rpy = "0 1.570796 0"/>
+            <origin xyz = "0 0 0.01" rpy = "0 0 0"/>
             <geometry>
-                <mesh filename = "file://$(find MRP_Description)/meshes/wheel_coupler_assembly.stl" scale = "0.001 0.001 0.001"/>
+                <cylinder length = '0.02' radius = '0.0925'/>
             </geometry>
         </collision>
         <inertial>
-            <mass value = "0.147595"/>
+            <mass value = "0.15"/>
             <inertia
-                        ixx = "${a * 3.20634763e-4}"
-                        ixy = "${a * 1e-6}"
-                        ixz = "${a * 1e-6}"
-                        iyy = "${a * 3.20634763e-4}"
-                        iyz = "${a * 1e-6}"
-                        izz = "${a * 6.314298594e-4}"/>
+                ixx = "${b * 3.20634763e-4}"
+                ixy = "${b * 1e-8}"
+                ixz = "${b * 1e-8}"
+                iyy = "${b * 3.20634763e-4}"
+                iyz = "${b * 1e-8}"
+                izz = "${b * 6.314298594e-4}"/>
         </inertial>
     </link>
+    <!-- rear right wheel to chassis joint -->
+    <joint name = 'rear_right_wheel_joint' type = 'continuous'>
+        <parent link = 'chassis_link'/>
+        <child link = 'rear_right_wheel'/>
+        <origin xyz = '-0.1355 -0.144 -0.0285' rpy = '1.570796 0 0'/>
+        <axis xyz = '0 0 -1'/>
+        <dynamics damping = '${d}' />
+    </joint>
     <!-- rear right wheel -->
     <link name = 'rear_right_wheel'>
@@ -276,23 +98,31 @@
                 <mesh filename = "file://$(find MRP_Description)/meshes/wheel_coupler_assembly.stl" scale = "0.001 0.001 0.001"/>
             </geometry>
-            <material name = 'grey'/>
+            <material name = 'purple'/>
         </visual>
         <collision>
-            <origin xyz = "0 0 0.012" rpy = "0 1.570796 0"/>
+            <origin xyz = "0 0 0.01" rpy = "0 0 0"/>
             <geometry>
-                <mesh filename = "file://$(find MRP_Description)/meshes/wheel_coupler_assembly.stl" scale = "0.001 0.001 0.001"/>
+                <cylinder length = '0.02' radius = '0.0925'/>
             </geometry>
         </collision>
         <inertial>
-            <mass value = "0.147595"/>
+            <mass value = "0.15"/>
             <inertia
-                        ixx = "${a * 3.20634763e-4}"
-                        ixy = "${a * 1e-6}"
-                        ixz = "${a * 1e-6}"
-                        iyy = "${a * 3.20634763e-4}"
-                        iyz = "${a * 1e-6}"
-                        izz = "${a * 6.314298594e-4}"/>
+                ixx = "${b * 3.20634763e-4}"
+                ixy = "${b * 1e-8}"
+                ixz = "${b * 1e-8}"
+                iyy = "${b * 3.20634763e-4}"
+                iyz = "${b * 1e-8}"
+                izz = "${b * 6.314298594e-4}"/>
         </inertial>
     </link>
+    <!-- front left wheel to chassis joint -->
+    <joint name = 'front_left_wheel_joint' type = 'continuous'>
+        <parent link = 'chassis_link'/>
+        <child link = 'front_left_wheel'/>
+        <origin xyz = '0.1755 0.144 -0.0285' rpy = '-1.570796 0 0'/>
+        <axis xyz = '0 0 1'/>
+        <dynamics damping = '${d}' />
+    </joint>
     <!-- front left wheel -->
     <link name = 'front_left_wheel'>
@@ -302,23 +132,31 @@
                 <mesh filename = "file://$(find MRP_Description)/meshes/wheel_coupler_assembly.stl" scale = "0.001 0.001 0.001"/>
             </geometry>
-            <material name = 'grey'/>
+            <material name = 'purple'/>
         </visual>
         <collision>
-            <origin xyz = "0 0 0.012" rpy = "0 1.570796 0"/>
+            <origin xyz = "0 0 0.01" rpy = "0 0 0"/>
             <geometry>
-                <mesh filename = "file://$(find MRP_Description)/meshes/wheel_coupler_assembly.stl" scale = "0.001 0.001 0.001"/>
+                <cylinder length = '0.02' radius = '0.0925'/>
             </geometry>
         </collision>
         <inertial>
-            <mass value = "0.147595"/>
+            <mass value = "0.15"/>
             <inertia
-                        ixx = "${a * 3.20634763e-4}"
-                        ixy = "${a * 1e-6}"
-                        ixz = "${a * 1e-6}"
-                        iyy = "${a * 3.20634763e-4}"
-                        iyz = "${a * 1e-6}"
-                        izz = "${a * 6.314298594e-4}"/>
+                ixx = "${b * 3.20634763e-4}"
+                ixy = "${b * 1e-8}"
+                ixz = "${b * 1e-8}"
+                iyy = "${b * 3.20634763e-4}"
+                iyz = "${b * 1e-8}"
+                izz = "${b * 6.314298594e-4}"/>
         </inertial>
     </link>
+    <!-- front right wheel to chassis joint -->
+    <joint name = 'front_right_wheel_joint' type = 'continuous'>
+        <parent link = 'chassis_link'/>
+        <child link = 'front_right_wheel'/>
+        <origin xyz = '0.1755 -0.144 -0.0285' rpy = '1.570796 0 0'/>
+        <axis xyz = '0 0 -1'/>
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
File: src/MRP_Description/urdf/MRP_Gazebo_Control.xacro (robot description, xacro)
@@ -6,8 +6,8 @@
             <num_wheel_pairs>2</num_wheel_pairs>
             <!-- wheels -->
-            <left_joint>RLM_RLW_joint</left_joint>
-            <left_joint>FLM_FLW_joint</left_joint>
-            <right_joint>RRM_RRW_joint</right_joint>
-            <right_joint>FRM_FRW_joint</right_joint>
+            <left_joint>rear_left_wheel_joint</left_joint>
+            <left_joint>front_left_wheel_joint</left_joint>
+            <right_joint>rear_right_wheel_joint</right_joint>
+            <right_joint>front_right_wheel_joint</right_joint>
             <!-- kinematics -->
             <wheel_separation> 0.288 </wheel_separation>

File: src/MRP_Description/urdf/MRP_Gazebo_Properties.xacro (robot description, xacro)
@@ -2,25 +2,9 @@
 <robot xmlns:xacro="http://www.ros.org/wiki/xacro">
     <!--                PROPERTIES:                 -->
-    <xacro:property name = 'mu1' value = '1.5'/>
-    <xacro:property name = 'mu2' value = '1.5'/>
+    <xacro:property name = 'mu1' value = '10'/>
+    <xacro:property name = 'mu2' value = '10'/>
     <!--                STRUCTURAL LINKS:                 -->
     <gazebo reference = 'chassis_link'>
         <material>Gazebo/Black</material>
-    </gazebo>
-    <gazebo reference = 'pendulum_bracket_link'>
-        <material>Gazebo/Black</material>
-    </gazebo>
-    <!--                MOTORS:                 -->
-    <gazebo reference = 'rear_left_motor'>
-        <material>Gazebo/Red</material>
-    </gazebo>
-    <gazebo reference = 'rear_right_motor'>
-        <material>Gazebo/Red</material>
-    </gazebo>
-    <gazebo reference = 'front_left_motor'>
-        <material>Gazebo/Red</material>
-    </gazebo>
-    <gazebo reference = 'front_right_motor'>
-        <material>Gazebo/Red</material>
     </gazebo>
     <!--                WHEELS:                 -->
@@ -44,4 +28,4 @@
         <mu1 value="${mu1}" />
         <mu2 value="${mu2}" />
-    </gazebo>
+    </gazebo>s
 </robot>
