Commit message: added inertias to the URDF

File: src/MRP_Description/urdf/MRP_Body.xacro (robot description, xacro)
@@ -23,5 +23,5 @@
         <parent link = 'chassis_link'/>
         <child link = 'rear_left_motor'/>
-        <origin xyz = '-0.1355 0.1015 -0.003'/>
+        <origin xyz = '-0.1355 0.1015 -0.003' rpy = '-1.570796 0 0'/>
     </joint>
     <!-- rear left wheel to rear left motor joint -->
@@ -29,6 +29,6 @@
         <parent link = 'rear_left_motor'/>
         <child link = 'rear_left_wheel'/>
-        <origin xyz = '0 0.0425 -0.0255'/>
-        <axis xyz = '0 1 0'/>
+        <origin xyz = '0 0.0255 0.0425' rpy = '0 0 0'/>
+        <axis xyz = '0 0 1'/>
     </joint>
     <!-- rear right wheel to rear right motor joint -->
@@ -36,6 +36,6 @@
         <parent link = 'rear_right_motor'/>
         <child link = 'rear_right_wheel'/>
-        <origin xyz = '0 -0.0425 -0.0255'/>
-        <axis xyz = '0 1 0'/>
+        <origin xyz = '0 -0.0255 0.0425' rpy = '0 0 0'/>
+        <axis xyz = '0 0 -1'/>
     </joint>
     <!-- rear right motor to chassis joint -->
@@ -43,5 +43,5 @@
         <parent link = 'chassis_link'/>
         <child link = 'rear_right_motor'/>
-        <origin xyz = '-0.1355 -0.1015 -0.003'/>
+        <origin xyz = '-0.1355 -0.1015 -0.003' rpy = '1.570796 0 0'/>
     </joint>
     <!-- chassis to pendulum bracket joint -->
@@ -57,5 +57,5 @@
         <parent link = 'pendulum_bracket_link'/>
         <child link = 'front_left_motor'/>
-        <origin xyz = '0 0.1015 -0.029438'/>
+        <origin xyz = '0 0.1015 -0.029438' rpy = '-1.570796 0 0'/>
     </joint>
     <!-- front left wheel to front left motor joint -->
@@ -63,6 +63,6 @@
         <parent link = 'front_left_motor'/>
         <child link = 'front_left_wheel'/>
-        <origin xyz = '0 0.0425 0.0115'/>
-        <axis xyz = '0 1 0'/>
+        <origin xyz = '0 -0.0115 0.0425' rpy = '0 0 0'/>
+        <axis xyz = '0 0 1'/>
     </joint>
     <!-- front right motor to pendulum bracket joint -->
@@ -70,5 +70,5 @@
         <parent link = 'pendulum_bracket_link'/>
         <child link = 'front_right_motor'/>
-        <origin xyz = '0 -0.1015 -0.029438'/>
+        <origin xyz = '0 -0.1015 -0.029438' rpy = '1.570796 0 0'/>
     </joint>
     <!-- front right wheel to front right motor joint -->
@@ -76,6 +76,6 @@
         <parent link = 'front_right_motor'/>
         <child link = 'front_right_wheel'/>
-        <origin xyz = '0 -0.0425 0.0115'/>
-        <axis xyz = '0 1 0'/>
+        <origin xyz = '0 0.0115 0.0425' rpy = '0 0 0'/>
+        <axis xyz = '0 0 -1'/>
     </joint>
     <!--                STRUCTURAL LINKS:                 -->
@@ -98,4 +98,8 @@
             </geometry>
         </collision>
+        <inertial>
+            <mass value = '0.27224'/>
+            <inertia ixx = '2.853307738e-3' ixy = '0' ixz = '0' iyy = '1.442962747e-3' iyz = '0' izz = '4.291733152e-3'/>
+        </inertial>
     </link>
     <!-- pendulum bracket link -->
@@ -114,4 +118,8 @@
             </geometry>
         </collision>
+        <inertial>
+            <mass value = '0.08492'/>
+            <inertia ixx = '3.682697333e-5' ixy = '0' ixz = '0' iyy = '4.670883067e-4' iyz = '0' izz = '4.685319467e-4'/>
+        </inertial>
     </link>
     <!--                MOTORS:                 -->
@@ -119,64 +127,80 @@
     <link name = 'rear_left_motor'>
         <visual>
-            <origin xyz = "0 0 -0.0185" rpy = "1.570796 0 3.141592"/>
-            <geometry>
-                <mesh filename = "file://$(find MRP_Description)/meshes/520_dc_gear_motor.stl" scale = "0.001 0.001 0.001"/>
-            </geometry>
-            <material name = 'red'/>
-        </visual>
-        <collision>
-            <origin xyz = "0 0 -0.0185" rpy = "1.570796 0 3.141592"/>
-            <geometry>
-                <mesh filename = "file://$(find MRP_Description)/meshes/520_dc_gear_motor.stl" scale = "0.001 0.001 0.001"/>
-            </geometry>
-        </collision>
+            <origin xyz = "0 0.0185 0 " rpy = "0 0 3.141592"/>
+            <geometry>
+                <mesh filename = "file://$(find MRP_Description)/meshes/520_dc_gear_motor.stl" scale = "0.001 0.001 0.001"/>
+            </geometry>
+            <material name = 'red'/>
+        </visual>
+        <collision>
+            <origin xyz = "0 0.0185 0" rpy = "0 0 3.141592"/>
+            <geometry>
+                <mesh filename = "file://$(find MRP_Description)/meshes/520_dc_gear_motor.stl" scale = "0.001 0.001 0.001"/>
+            </geometry>
+        </collision>
+        <inertial>
+            <mass value = '0.1579'/>
+            <inertia ixx = '5.188001875e-5' ixy = '0' ixz = '0' iyy = '5.188001875e-5' iyz = '0' izz = '2.70206375e-5'/>
+        </inertial>
     </link>
     <!-- rear right motor link -->
     <link name = 'rear_right_motor'>
         <visual>
-            <origin xyz = "0 0 -0.0185" rpy = "1.570796 0 0"/>
-            <geometry>
-                <mesh filename = "file://$(find MRP_Description)/meshes/520_dc_gear_motor.stl" scale = "0.001 0.001 0.001"/>
-            </geometry>
-            <material name = 'red'/>
-        </visual>
-        <collision>
-            <origin xyz = "0 0 -0.0185" rpy = "1.570796 0 0"/>
-            <geometry>
-                <mesh filename = "file://$(find MRP_Description)/meshes/520_dc_gear_motor.stl" scale = "0.001 0.001 0.001"/>
-            </geometry>
-        </collision>
+            <origin xyz = "0 -0.0185 0" rpy = "0 0 0"/>
+            <geometry>
+                <mesh filename = "file://$(find MRP_Description)/meshes/520_dc_gear_motor.stl" scale = "0.001 0.001 0.001"/>
+            </geometry>
+            <material name = 'red'/>
+        </visual>
+        <collision>
+            <origin xyz = "0 -0.0185 0" rpy = "0 0 0"/>
+            <geometry>
+                <mesh filename = "file://$(find MRP_Description)/meshes/520_dc_gear_motor.stl" scale = "0.001 0.001 0.001"/>
+            </geometry>
+        </collision>
+        <inertial>
+            <mass value = '0.1579'/>
+            <inertia ixx = '5.188001875e-5' ixy = '0' ixz = '0' iyy = '5.188001875e-5' iyz = '0' izz = '2.70206375e-5'/>
+        </inertial>
     </link>
     <!-- front left motor -->
     <link name = 'front_left_motor'>
         <visual>
-            <origin xyz = "0 0 0.0185" rpy = "1.570796 0 3.141592"/>
-            <geometry>
-                <mesh filename = "file://$(find MRP_Description)/meshes/520_dc_gear_motor.stl" scale = "0.001 0.001 0.001"/>
-            </geometry>
-            <material name = 'red'/>
-        </visual>
-        <collision>
-            <origin xyz = "0 0 0.0185" rpy = "1.570796 0 3.141592"/>
-            <geometry>
-                <mesh filename = "file://$(find MRP_Description)/meshes/520_dc_gear_motor.stl" scale = "0.001 0.001 0.001"/>
-            </geometry>
-        </collision>
+            <origin xyz = "0 -0.0185 0" rpy = "0 0 3.141592"/>
+            <geometry>
+                <mesh filename = "file://$(find MRP_Description)/meshes/520_dc_gear_motor.stl" scale = "0.001 0.001 0.001"/>
+            </geometry>
+            <material name = 'red'/>
+        </visual>
+        <collision>
+            <origin xyz = "0 -0.0185 0" rpy = "0 0 3.141592"/>
+            <geometry>
+                <mesh filename = "file://$(find MRP_Description)/meshes/520_dc_gear_motor.stl" scale = "0.001 0.001 0.001"/>
+            </geometry>
+        </collision>
+        <inertial>
+            <mass value = '0.1579'/>
+            <inertia ixx = '5.188001875e-5' ixy = '0' ixz = '0' iyy = '5.188001875e-5' iyz = '0' izz = '2.70206375e-5'/>
+        </inertial>
     </link>
     <!-- front right motor -->
     <link name = 'front_right_motor'>
         <visual>
-            <origin xyz = "0 0 0.0185" rpy = "1.570796 0 0"/>
-            <geometry>
-                <mesh filename = "file://$(find MRP_Description)/meshes/520_dc_gear_motor.stl" scale = "0.001 0.001 0.001"/>
-            </geometry>
-            <material name = 'red'/>
-        </visual>
-        <collision>
-            <origin xyz = "0 0 0.0185" rpy = "1.570796 0 0"/>
-            <geometry>
-                <mesh filename = "file://$(find MRP_Description)/meshes/520_dc_gear_motor.stl" scale = "0.001 0.001 0.001"/>
-            </geometry>
-        </collision>
+            <origin xyz = "0 0.0185 0" rpy = "0 0 0"/>
+            <geometry>
+                <mesh filename = "file://$(find MRP_Description)/meshes/520_dc_gear_motor.stl" scale = "0.001 0.001 0.001"/>
+            </geometry>
+            <material name = 'red'/>
+        </visual>
+        <collision>
+            <origin xyz = "0 0.0185 0" rpy = "0 0 0"/>
+            <geometry>
+                <mesh filename = "file://$(find MRP_Description)/meshes/520_dc_gear_motor.stl" scale = "0.001 0.001 0.001"/>
+            </geometry>
+        </collision>
+        <inertial>
+            <mass value = '0.1579'/>
+            <inertia ixx = '5.188001875e-5' ixy = '0' ixz = '0' iyy = '5.188001875e-5' iyz = '0' izz = '2.70206375e-5'/>
+        </inertial>
     </link>
     <!--                WHEELS:                 -->
@@ -184,20 +208,19 @@
     <link name = 'rear_left_wheel'>
         <visual>
-            <origin xyz = "0 0.012 0" rpy = "1.570796 0 -1.570796"/>
-            <geometry>
-                <mesh filename = "file://$(find MRP_Description)/meshes/wheel_coupler_assembly.stl" scale = "0.001 0.001 0.001"/>
-            </geometry>
-            <material name = 'grey'/>
-        </visual>
-        <collision>
-            <origin xyz = "0 0.012 0" rpy = "1.570796 0 -1.570796"/>
-            <geometry>
-                <mesh filename = "file://$(find MRP_Description)/meshes/wheel_coupler_assembly.stl" scale = "0.001 0.001 0.001"/>
-            </geometry>
-        </collision>
-        <inertial>
-            <mass value = "0.15"/>
-            <inertia ixx="0.028564013" ixy="-0.000252573" ixz="-0.000026632"
-            iyy="0.000671702" iyz="-0.002904292" izz="0.027909635"/>
+            <origin xyz = "0 0 0.012" rpy = "0 1.570796 0"/>
+            <geometry>
+                <mesh filename = "file://$(find MRP_Description)/meshes/wheel_coupler_assembly.stl" scale = "0.001 0.001 0.001"/>
+            </geometry>
+            <material name = 'grey'/>
+        </visual>
+        <collision>
+            <origin xyz = "0 0 0.012" rpy = "0 1.570796 0"/>
+            <geometry>
+                <mesh filename = "file://$(find MRP_Description)/meshes/wheel_coupler_assembly.stl" scale = "0.001 0.001 0.001"/>
+            </geometry>
+        </collision>
+        <inertial>
+            <mass value = "0.147595"/>
+            <inertia ixx="3.20634763e-4" ixy="0" ixz="0" iyy="3.20634763e-4" iyz="0" izz="6.314298594e-4"/>
         </inertial>
     </link>
@@ -205,20 +228,19 @@
     <link name = 'rear_right_wheel'>
         <visual>
-            <origin xyz = "0 -0.012 0" rpy = "1.570796 0 1.570796"/>
-            <geometry>
-                <mesh filename = "file://$(find MRP_Description)/meshes/wheel_coupler_assembly.stl" scale = "0.001 0.001 0.001"/>
-            </geometry>
-            <material name = 'grey'/>
-        </visual>
-        <collision>
-            <origin xyz = "0 -0.012 0" rpy = "1.570796 0 1.570796"/>
-            <geometry>
-                <mesh filename = "file://$(find MRP_Description)/meshes/wheel_coupler_assembly.stl" scale = "0.001 0.001 0.001"/>
-            </geometry>
-        </collision>
-        <inertial>
-            <mass value = "0.15"/>
-            <inertia ixx="0.028564013" ixy="-0.000252573" ixz="-0.000026632"
-            iyy="0.000671702" iyz="-0.002904292" izz="0.027909635"/>
+            <origin xyz = "0 0 0.012" rpy = "0 1.570796 0"/>
+            <geometry>
+                <mesh filename = "file://$(find MRP_Description)/meshes/wheel_coupler_assembly.stl" scale = "0.001 0.001 0.001"/>
+            </geometry>
+            <material name = 'grey'/>
+        </visual>
+        <collision>
+            <origin xyz = "0 0 0.012" rpy = "0 1.570796 0"/>
+            <geometry>
+                <mesh filename = "file://$(find MRP_Description)/meshes/wheel_coupler_assembly.stl" scale = "0.001 0.001 0.001"/>
+            </geometry>
+        </collision>
+        <inertial>
+            <mass value = "0.147595"/>
+            <inertia ixx="3.20634763e-4" ixy="0" ixz="0" iyy="3.20634763e-4" iyz="0" izz="6.314298594e-4"/>
         </inertial>
     </link>
@@ -226,41 +248,39 @@
     <link name = 'front_left_wheel'>
         <visual>
-            <origin xyz = "0 0.012 0" rpy = "1.570796 0 -1.570796"/>
-            <geometry>
-                <mesh filename = "file://$(find MRP_Description)/meshes/wheel_coupler_assembly.stl" scale = "0.001 0.001 0.001"/>
-            </geometry>
-            <material name = 'grey'/>
-        </visual>
-        <collision>
-            <origin xyz = "0 0.012 0" rpy = "1.570796 0 -1.570796"/>
-            <geometry>
-                <mesh filename = "file://$(find MRP_Description)/meshes/wheel_coupler_assembly.stl" scale = "0.001 0.001 0.001"/>
-            </geometry>
-        </collision>
-        <inertial>
-            <mass value = "0.15"/>
-            <inertia ixx="0.028564013" ixy="-0.000252573" ixz="-0.000026632"
-            iyy="0.000671702" iyz="-0.002904292" izz="0.027909635"/>
-        </inertial>
-    </link>
-    <!-- front left wheel -->
+            <origin xyz = "0 0 0.012" rpy = "0 1.570796 0"/>
+            <geometry>
+                <mesh filename = "file://$(find MRP_Description)/meshes/wheel_coupler_assembly.stl" scale = "0.001 0.001 0.001"/>
+            </geometry>
+            <material name = 'grey'/>
+        </visual>
+        <collision>
+            <origin xyz = "0 0 0.012" rpy = "0 1.570796 0"/>
+            <geometry>
+                <mesh filename = "file://$(find MRP_Description)/meshes/wheel_coupler_assembly.stl" scale = "0.001 0.001 0.001"/>
+            </geometry>
+        </collision>
+        <inertial>
+            <mass value = "0.147595"/>
+            <inertia ixx="3.20634763e-4" ixy="0" ixz="0" iyy="3.20634763e-4" iyz="0" izz="6.314298594e-4"/>
+        </inertial>
+    </link>
+    <!-- front right wheel -->
     <link name = 'front_right_wheel'>
         <visual>
-            <origin xyz = "0 -0.012 0" rpy = "1.570796 0 1.570796"/>
-            <geometry>
-                <mesh filename = "file://$(find MRP_Description)/meshes/wheel_coupler_assembly.stl" scale = "0.001 0.001 0.001"/>
-            </geometry>
-            <material name = 'grey'/>
-        </visual>
-        <collision>
-            <origin xyz = "0 -0.012 0" rpy = "1.570796 0 1.570796"/>
-            <geometry>
-                <mesh filename = "file://$(find MRP_Description)/meshes/wheel_coupler_assembly.stl" scale = "0.001 0.001 0.001"/>
-            </geometry>
-        </collision>
-        <inertial>
-            <mass value = "0.15"/>
-            <inertia ixx="0.028564013" ixy="-0.000252573" ixz="-0.000026632"
-            iyy="0.000671702" iyz="-0.002904292" izz="0.027909635"/>
+            <origin xyz = "0 0 0.012" rpy = "0 1.570796 0"/>
+            <geometry>
+                <mesh filename = "file://$(find MRP_Description)/meshes/wheel_coupler_assembly.stl" scale = "0.001 0.001 0.001"/>
+            </geometry>
+            <material name = 'grey'/>
+        </visual>
+        <collision>
+            <origin xyz = "0 0 0.012" rpy = "0 1.570796 0"/>
+            <geometry>
+                <mesh filename = "file://$(find MRP_Description)/meshes/wheel_coupler_assembly.stl" scale = "0.001 0.001 0.001"/>
+            </geometry>
+        </collision>
+        <inertial>
+            <mass value = "0.147595"/>
+            <inertia ixx="3.20634763e-4" ixy="0" ixz="0" iyy="3.20634763e-4" iyz="0" izz="6.314298594e-4"/>
         </inertial>
     </link>

Commit message: messed around with old URDF model

File: src/MRP_Description/urdf/MRP_Body.xacro (robot description, xacro)
@@ -3,5 +3,5 @@
 <robot xmlns:xacro="http://www.ros.org/wiki/xacro">
     <!--                PROPERTIES:                 -->
-    <xacro:property name='a' value='4'/>
+    <xacro:property name='a' value='6'/>
     <material name = "black">
         <color rgba = "0.1 0.1 0.1 1"/>

File: src/MRP_Description/urdf/MRP_Gazebo_Properties.xacro (robot description, xacro)
@@ -2,6 +2,6 @@
 <robot xmlns:xacro="http://www.ros.org/wiki/xacro">
     <!--                PROPERTIES:                 -->
-    <xacro:property name = 'mu1' value = '1.0'/>
-    <xacro:property name = 'mu2' value = '1.0'/>
+    <xacro:property name = 'mu1' value = '1.5'/>
+    <xacro:property name = 'mu2' value = '1.5'/>
     <!--                STRUCTURAL LINKS:                 -->
     <gazebo reference = 'chassis_link'>

Commit message: modeled collision of wheels as spheres to permit proper turning in place

File: src/MRP_Description/urdf/MRP_Body.xacro (robot description, xacro)
@@ -69,5 +69,6 @@
             <origin xyz = "0 0 0.01" rpy = "0 0 0"/>
             <geometry>
-                <cylinder length = '0.02' radius = '0.0925'/>
+                <!-- <cylinder length = '0.02' radius = '0.0925'/> -->
+                <sphere radius = '0.0925'/>
             </geometry>
         </collision>
@@ -103,5 +104,6 @@
             <origin xyz = "0 0 0.01" rpy = "0 0 0"/>
             <geometry>
-                <cylinder length = '0.02' radius = '0.0925'/>
+                <!-- <cylinder length = '0.02' radius = '0.0925'/> -->
+                <sphere radius = '0.0925'/>
             </geometry>
         </collision>
@@ -137,5 +139,6 @@
             <origin xyz = "0 0 0.01" rpy = "0 0 0"/>
             <geometry>
-                <cylinder length = '0.02' radius = '0.0925'/>
+                <!-- <cylinder length = '0.02' radius = '0.0925'/> -->
+                <sphere radius = '0.0925'/>
             </geometry>
         </collision>
@@ -171,5 +174,6 @@
             <origin xyz = "0 0 0.01" rpy = "0 0 0"/>
             <geometry>
-                <cylinder length = '0.02' radius = '0.0925'/>
+                <!-- <cylinder length = '0.02' radius = '0.0925'/> -->
+                <sphere radius = '0.0925'/>
             </geometry>
         </collision>

Commit message: reduced the damping on the joints -> saw improved performance in simulation

File: src/MRP_Description/urdf/MRP_Body.xacro (robot description, xacro)
@@ -4,5 +4,5 @@
     <xacro:property name = 'a' value = '1'/>
     <xacro:property name = 'b' value = '4'/>
-    <xacro:property name = 'd' value = '0.2'/>
+    <xacro:property name = 'd' value = '0.02'/>
     <material name = "black">
         <color rgba = "0.1 0.1 0.1 1"/>

Commit message: urdf tweaks

File: src/MRP_Description/urdf/MRP_Body.xacro (robot description, xacro)
@@ -4,5 +4,5 @@
     <xacro:property name = 'a' value = '1'/>
     <xacro:property name = 'b' value = '4'/>
-    <xacro:property name = 'd' value = '0.02'/>
+    <xacro:property name = 'd' value = '0.05'/>
     <material name = "black">
         <color rgba = "0.1 0.1 0.1 1"/>
@@ -12,5 +12,9 @@
     </material>
     <material name = "purple">
-        <color rgba = "0.25 0.15 0.25 1"/>
+        <!-- <color rgba = "0.25 0.15 0.25 1"/> -->
+        <color rgba="0.56 0.0 1.0 1.0"/>
+    </material>
+    <material name = 'light gray'>
+        <color rgba="0.83 0.83 0.83 1.0"/>
     </material>
     <!-- base link -->
@@ -30,5 +34,5 @@
                 <mesh filename = "file://$(find MRP_Description)/meshes/entire_chassis.stl" scale = "0.001 0.001 0.001"/>
             </geometry>
-            <material name = 'black'/>
+            <material name = 'light gray'/>
         </visual>
         <collision>
@@ -69,6 +73,6 @@
             <origin xyz = "0 0 0.01" rpy = "0 0 0"/>
             <geometry>
-                <!-- <cylinder length = '0.02' radius = '0.0925'/> -->
-                <sphere radius = '0.0925'/>
+                <cylinder length = '0.02' radius = '0.0925'/>
+                <!-- <sphere radius = '0.0925'/> -->
             </geometry>
         </collision>
@@ -104,6 +108,6 @@
             <origin xyz = "0 0 0.01" rpy = "0 0 0"/>
             <geometry>
-                <!-- <cylinder length = '0.02' radius = '0.0925'/> -->
-                <sphere radius = '0.0925'/>
+                <cylinder length = '0.02' radius = '0.0925'/>
+                <!-- <sphere radius = '0.0925'/> -->
             </geometry>
         </collision>
@@ -139,6 +143,6 @@
             <origin xyz = "0 0 0.01" rpy = "0 0 0"/>
             <geometry>
-                <!-- <cylinder length = '0.02' radius = '0.0925'/> -->
-                <sphere radius = '0.0925'/>
+                <cylinder length = '0.02' radius = '0.0925'/>
+                <!-- <sphere radius = '0.0925'/> -->
             </geometry>
         </collision>
@@ -174,6 +178,6 @@
             <origin xyz = "0 0 0.01" rpy = "0 0 0"/>
             <geometry>
-                <!-- <cylinder length = '0.02' radius = '0.0925'/> -->
-                <sphere radius = '0.0925'/>
+                <cylinder length = '0.02' radius = '0.0925'/>
+                <!-- <sphere radius = '0.0925'/> -->
             </geometry>
         </collision>

File: src/MRP_Description/urdf/MRP_Gazebo_Properties.xacro (robot description, xacro)
@@ -2,6 +2,6 @@
 <robot xmlns:xacro="http://www.ros.org/wiki/xacro">
     <!--                PROPERTIES                 -->
-    <xacro:property name = 'mu1' value = '1'/>
-    <xacro:property name = 'mu2' value = '1'/>
+    <xacro:property name = 'mu1' value = '0.5'/>
+    <xacro:property name = 'mu2' value = '0.5'/>
     <!--                STRUCTURAL LINKS                 -->
     <gazebo reference = 'chassis_link'>
