Commit message: changed mesh filepath to be independent from machine

File: src/MRP_Description/urdf/MRP_Body.xacro (robot description, xacro)
@@ -32,5 +32,6 @@
             <origin xyz = '0 0 0' rpy = '1.570796 0 0'/>
             <geometry>
-                <mesh filename = "file://$(find MRP_Description)/meshes/entire_chassis.stl" scale = "0.001 0.001 0.001"/>
+                <!-- <mesh filename = "file://$(find MRP_Description)/meshes/entire_chassis.stl" scale = "0.001 0.001 0.001"/> -->
+                <mesh filename = "package://MRP_Description/meshes/entire_chassis.stl" scale = "0.001 0.001 0.001"/>
             </geometry>
             <material name = 'light gray'/>
@@ -66,5 +67,6 @@
             <origin xyz = "0 0 0.012" rpy = "0 1.570796 0"/>
             <geometry>
-                <mesh filename = "file://$(find MRP_Description)/meshes/wheel_coupler_assembly.stl" scale = "0.001 0.001 0.001"/>
+                <!-- <mesh filename = "file://$(find MRP_Description)/meshes/wheel_coupler_assembly.stl" scale = "0.001 0.001 0.001"/> -->
+                <mesh filename = "package://MRP_Description/meshes/wheel_coupler_assembly.stl" scale = "0.001 0.001 0.001"/>
             </geometry>
             <material name = 'purple'/>
@@ -101,5 +103,6 @@
             <origin xyz = "0 0 0.012" rpy = "0 1.570796 0"/>
             <geometry>
-                <mesh filename = "file://$(find MRP_Description)/meshes/wheel_coupler_assembly.stl" scale = "0.001 0.001 0.001"/>
+                <!-- <mesh filename = "file://$(find MRP_Description)/meshes/wheel_coupler_assembly.stl" scale = "0.001 0.001 0.001"/> -->
+                <mesh filename = "package://MRP_Description/meshes/wheel_coupler_assembly.stl" scale = "0.001 0.001 0.001"/>
             </geometry>
             <material name = 'purple'/>
@@ -136,5 +139,6 @@
             <origin xyz = "0 0 0.012" rpy = "0 1.570796 0"/>
             <geometry>
-                <mesh filename = "file://$(find MRP_Description)/meshes/wheel_coupler_assembly.stl" scale = "0.001 0.001 0.001"/>
+                <!-- <mesh filename = "file://$(find MRP_Description)/meshes/wheel_coupler_assembly.stl" scale = "0.001 0.001 0.001"/> -->
+                <mesh filename = "package://MRP_Description/meshes/wheel_coupler_assembly.stl" scale = "0.001 0.001 0.001"/>
             </geometry>
             <material name = 'purple'/>
@@ -171,5 +175,6 @@
             <origin xyz = "0 0 0.012" rpy = "0 1.570796 0"/>
             <geometry>
-                <mesh filename = "file://$(find MRP_Description)/meshes/wheel_coupler_assembly.stl" scale = "0.001 0.001 0.001"/>
+                <!-- <mesh filename = "file://$(find MRP_Description)/meshes/wheel_coupler_assembly.stl" scale = "0.001 0.001 0.001"/> -->
+                <mesh filename = "package://MRP_Description/meshes/wheel_coupler_assembly.stl" scale = "0.001 0.001 0.001"/>
             </geometry>
             <material name = 'purple'/>
