Commit message: modified plugin to reflect 4-wheeled robot

File: src/MRP_Hardware_Interface/description/ros2_control/diffbot.ros2_control.xacro (robot description, xacro)
@@ -1,25 +1,33 @@
 <?xml version="1.0"?>
 <robot xmlns:xacro="http://www.ros.org/wiki/xacro">
-  <xacro:macro name="diffbot_ros2_control" params="name prefix use_mock_hardware">
+  <xacro:macro name="diffbot_ros2_control" params="name prefix">
     <ros2_control name="${name}" type="system">
-      <xacro:unless value="${use_mock_hardware}">
-        <hardware>
-          <plugin>ros2_control_demo_example_2/DiffBotSystemHardware</plugin>
-          <param name="example_param_hw_start_duration_sec">0</param>
-          <param name="example_param_hw_stop_duration_sec">3.0</param>
-        </hardware>
-      </xacro:unless>
-      <xacro:if value="${use_mock_hardware}">
-        <hardware>
-          <plugin>mock_components/GenericSystem</plugin>
-          <param name="calculate_dynamics">true</param>
-        </hardware>
-      </xacro:if>
-      <joint name="${prefix}left_wheel_joint">
+      <hardware>
+        <plugin>MRP_Hardware_Interface/DiffBotSystemHardware</plugin>
+        <param name="front_left_wheel_name">front_left_wheel_joint</param>
+        <param name="front_right_wheel_name">front_right_wheel_joint</param>
+        <param name="rear_left_wheel_name">rear_left_wheel_joint</param>
+        <param name="rear_right_wheel_name">rear_right_wheel_joint</param>
+        <param name="device">/dev/serial/by-path/platform-fd500000.pcie-pci-0000:01:00.0-usb-0:1.3:1.0</param>
+        <param name="baud_rate">57600</param>
+        <param name="timeout_ms">1000</param>
+        <param name="enc_counts_per_rev">1320</param>
+      </hardware>
+      <joint name="${prefix}front_left_wheel_joint">
         <command_interface name="velocity"/>
         <state_interface name="position"/>
         <state_interface name="velocity"/>
       </joint>
-      <joint name="${prefix}right_wheel_joint">
+      <joint name="${prefix}front_right_wheel_joint">
+        <command_interface name="velocity"/>
+        <state_interface name="position"/>
+        <state_interface name="velocity"/>
+      </joint>
+      <joint name="${prefix}rear_left_wheel_joint">
+        <command_interface name="velocity"/>
+        <state_interface name="position"/>
+        <state_interface name="velocity"/>
+      </joint>
+      <joint name="${prefix}rear_right_wheel_joint">
         <command_interface name="velocity"/>
         <state_interface name="position"/>
