Commit message: package:// was breaking gazebo. idk how it will work for robot_description on different devices

File: src/mrp_description/urdf/MRP_Body.xacro (robot description, xacro)
@@ -32,6 +32,6 @@
             <origin xyz = '0 0 0' rpy = '1.570796 0 0'/>
             <geometry>
-                <!-- <mesh filename = "file://$(find mrp_description)/meshes/entire_chassis.stl" scale = "0.001 0.001 0.001"/> -->
-                <mesh filename = "package://mrp_description/meshes/entire_chassis.stl" scale = "0.001 0.001 0.001"/>
+                <mesh filename = "file://$(find mrp_description)/meshes/entire_chassis.stl" scale = "0.001 0.001 0.001"/>
+                <!-- <mesh filename = "package://mrp_description/meshes/entire_chassis.stl" scale = "0.001 0.001 0.001"/> -->
             </geometry>
             <material name = 'light gray'/>
@@ -67,6 +67,6 @@
             <origin xyz = "0 0 0.012" rpy = "0 1.570796 0"/>
             <geometry>
-                <!-- <mesh filename = "file://$(find mrp_description)/meshes/wheel_coupler_assembly.stl" scale = "0.001 0.001 0.001"/> -->
-                <mesh filename = "package://mrp_description/meshes/wheel_coupler_assembly.stl" scale = "0.001 0.001 0.001"/>
+                <mesh filename = "file://$(find mrp_description)/meshes/wheel_coupler_assembly.stl" scale = "0.001 0.001 0.001"/>
+                <!-- <mesh filename = "package://mrp_description/meshes/wheel_coupler_assembly.stl" scale = "0.001 0.001 0.001"/> -->
             </geometry>
             <material name = 'purple'/>
@@ -103,6 +103,6 @@
             <origin xyz = "0 0 0.012" rpy = "0 1.570796 0"/>
             <geometry>
-                <!-- <mesh filename = "file://$(find mrp_description)/meshes/wheel_coupler_assembly.stl" scale = "0.001 0.001 0.001"/> -->
-                <mesh filename = "package://mrp_description/meshes/wheel_coupler_assembly.stl" scale = "0.001 0.001 0.001"/>
+                <mesh filename = "file://$(find mrp_description)/meshes/wheel_coupler_assembly.stl" scale = "0.001 0.001 0.001"/>
+                <!-- <mesh filename = "package://mrp_description/meshes/wheel_coupler_assembly.stl" scale = "0.001 0.001 0.001"/> -->
             </geometry>
             <material name = 'purple'/>
@@ -139,6 +139,6 @@
             <origin xyz = "0 0 0.012" rpy = "0 1.570796 0"/>
             <geometry>
-                <!-- <mesh filename = "file://$(find mrp_description)/meshes/wheel_coupler_assembly.stl" scale = "0.001 0.001 0.001"/> -->
-                <mesh filename = "package://mrp_description/meshes/wheel_coupler_assembly.stl" scale = "0.001 0.001 0.001"/>
+                <mesh filename = "file://$(find mrp_description)/meshes/wheel_coupler_assembly.stl" scale = "0.001 0.001 0.001"/>
+                <!-- <mesh filename = "package://mrp_description/meshes/wheel_coupler_assembly.stl" scale = "0.001 0.001 0.001"/>    -->
             </geometry>
             <material name = 'purple'/>
@@ -175,6 +175,6 @@
             <origin xyz = "0 0 0.012" rpy = "0 1.570796 0"/>
             <geometry>
-                <!-- <mesh filename = "file://$(find mrp_description)/meshes/wheel_coupler_assembly.stl" scale = "0.001 0.001 0.001"/> -->
-                <mesh filename = "package://mrp_description/meshes/wheel_coupler_assembly.stl" scale = "0.001 0.001 0.001"/>
+                <mesh filename = "file://$(find mrp_description)/meshes/wheel_coupler_assembly.stl" scale = "0.001 0.001 0.001"/>
+                <!-- <mesh filename = "package://mrp_description/meshes/wheel_coupler_assembly.stl" scale = "0.001 0.001 0.001"/>  -->
             </geometry>
             <material name = 'purple'/>
