Commit message: doubled friction

File: src/mrp_description/urdf/MRP_Gazebo_Properties.xacro (robot description, xacro)
@@ -2,6 +2,6 @@
 <robot xmlns:xacro="http://www.ros.org/wiki/xacro">
     <!--                PROPERTIES                 -->
-    <xacro:property name = 'mu1' value = '0.5'/>
-    <xacro:property name = 'mu2' value = '0.5'/>
+    <xacro:property name = 'mu1' value = '1.0'/>
+    <xacro:property name = 'mu2' value = '1.0'/>
     <!--                STRUCTURAL LINKS                 -->
     <gazebo reference = 'chassis_link'>
