Commit message: fixed path to mesh

File: src/mrp_real_robot/urdf/MRP_Body.xacro (robot description, xacro)
@@ -32,6 +32,6 @@
             <origin xyz = '0 0 0' rpy = '1.570796 0 0'/>
             <geometry>
-                <!-- <mesh filename = "file://$(find MRP_Description)/meshes/entire_chassis.stl" scale = "0.001 0.001 0.001"/> -->
-                <mesh filename = "package://MRP_Description/meshes/entire_chassis.stl" scale = "0.001 0.001 0.001"/>
+                <mesh filename = "file://$(find mrp_real_robot)/meshes/entire_chassis.stl" scale = "0.001 0.001 0.001"/>
+                <!-- <mesh filename = "package://MRP_Description/meshes/entire_chassis.stl" scale = "0.001 0.001 0.001"/> -->
             </geometry>
             <material name = 'light gray'/>
@@ -67,6 +67,6 @@
             <origin xyz = "0 0 0.012" rpy = "0 1.570796 0"/>
             <geometry>
-                <!-- <mesh filename = "file://$(find MRP_Description)/meshes/wheel_coupler_assembly.stl" scale = "0.001 0.001 0.001"/> -->
-                <mesh filename = "package://MRP_Description/meshes/wheel_coupler_assembly.stl" scale = "0.001 0.001 0.001"/>
+                <mesh filename = "file://$(find mrp_real_robot)/meshes/wheel_coupler_assembly.stl" scale = "0.001 0.001 0.001"/>
+                <!-- <mesh filename = "package://MRP_Description/meshes/wheel_coupler_assembly.stl" scale = "0.001 0.001 0.001"/> -->
             </geometry>
             <material name = 'purple'/>
@@ -103,6 +103,6 @@
             <origin xyz = "0 0 0.012" rpy = "0 1.570796 0"/>
             <geometry>
-                <!-- <mesh filename = "file://$(find MRP_Description)/meshes/wheel_coupler_assembly.stl" scale = "0.001 0.001 0.001"/> -->
-                <mesh filename = "package://MRP_Description/meshes/wheel_coupler_assembly.stl" scale = "0.001 0.001 0.001"/>
+                <mesh filename = "file://$(find mrp_real_robot)/meshes/wheel_coupler_assembly.stl" scale = "0.001 0.001 0.001"/>
+                <!-- <mesh filename = "package://MRP_Description/meshes/wheel_coupler_assembly.stl" scale = "0.001 0.001 0.001"/> -->
             </geometry>
             <material name = 'purple'/>
@@ -139,6 +139,6 @@
             <origin xyz = "0 0 0.012" rpy = "0 1.570796 0"/>
             <geometry>
-                <!-- <mesh filename = "file://$(find MRP_Description)/meshes/wheel_coupler_assembly.stl" scale = "0.001 0.001 0.001"/> -->
-                <mesh filename = "package://MRP_Description/meshes/wheel_coupler_assembly.stl" scale = "0.001 0.001 0.001"/>
+                <mesh filename = "file://$(find mrp_real_robot)/meshes/wheel_coupler_assembly.stl" scale = "0.001 0.001 0.001"/>
+                <!-- <mesh filename = "package://MRP_Description/meshes/wheel_coupler_assembly.stl" scale = "0.001 0.001 0.001"/>    -->
             </geometry>
             <material name = 'purple'/>
@@ -175,6 +175,6 @@
             <origin xyz = "0 0 0.012" rpy = "0 1.570796 0"/>
             <geometry>
-                <!-- <mesh filename = "file://$(find MRP_Description)/meshes/wheel_coupler_assembly.stl" scale = "0.001 0.001 0.001"/> -->
-                <mesh filename = "package://MRP_Description/meshes/wheel_coupler_assembly.stl" scale = "0.001 0.001 0.001"/>
+                <mesh filename = "file://$(find mrp_real_robot)/meshes/wheel_coupler_assembly.stl" scale = "0.001 0.001 0.001"/>
+                <!-- <mesh filename = "package://MRP_Description/meshes/wheel_coupler_assembly.stl" scale = "0.001 0.001 0.001"/>  -->
             </geometry>
             <material name = 'purple'/>

Commit message: switched back to file:// from package://

File: src/mrp_real_robot/urdf/MRP_Body.xacro (robot description, xacro)
@@ -33,5 +33,5 @@
             <geometry>
                 <mesh filename = "file://$(find mrp_real_robot)/meshes/entire_chassis.stl" scale = "0.001 0.001 0.001"/>
-                <!-- <mesh filename = "package://MRP_Description/meshes/entire_chassis.stl" scale = "0.001 0.001 0.001"/> -->
+                <!-- <mesh filename = "package://mrp_real_robot/meshes/entire_chassis.stl" scale = "0.001 0.001 0.001"/> -->
             </geometry>
             <material name = 'light gray'/>
@@ -68,5 +68,5 @@
             <geometry>
                 <mesh filename = "file://$(find mrp_real_robot)/meshes/wheel_coupler_assembly.stl" scale = "0.001 0.001 0.001"/>
-                <!-- <mesh filename = "package://MRP_Description/meshes/wheel_coupler_assembly.stl" scale = "0.001 0.001 0.001"/> -->
+                <!-- <mesh filename = "package://mrp_real_robot/meshes/wheel_coupler_assembly.stl" scale = "0.001 0.001 0.001"/> -->
             </geometry>
             <material name = 'purple'/>
@@ -104,5 +104,5 @@
             <geometry>
                 <mesh filename = "file://$(find mrp_real_robot)/meshes/wheel_coupler_assembly.stl" scale = "0.001 0.001 0.001"/>
-                <!-- <mesh filename = "package://MRP_Description/meshes/wheel_coupler_assembly.stl" scale = "0.001 0.001 0.001"/> -->
+                <!-- <mesh filename = "package://mrp_real_robot/meshes/wheel_coupler_assembly.stl" scale = "0.001 0.001 0.001"/> -->
             </geometry>
             <material name = 'purple'/>
@@ -140,5 +140,5 @@
             <geometry>
                 <mesh filename = "file://$(find mrp_real_robot)/meshes/wheel_coupler_assembly.stl" scale = "0.001 0.001 0.001"/>
-                <!-- <mesh filename = "package://MRP_Description/meshes/wheel_coupler_assembly.stl" scale = "0.001 0.001 0.001"/>    -->
+                <!-- <mesh filename = "package://mrp_real_robot/meshes/wheel_coupler_assembly.stl" scale = "0.001 0.001 0.001"/>    -->
             </geometry>
             <material name = 'purple'/>
@@ -176,5 +176,5 @@
             <geometry>
                 <mesh filename = "file://$(find mrp_real_robot)/meshes/wheel_coupler_assembly.stl" scale = "0.001 0.001 0.001"/>
-                <!-- <mesh filename = "package://MRP_Description/meshes/wheel_coupler_assembly.stl" scale = "0.001 0.001 0.001"/>  -->
+                <!-- <mesh filename = "package://mrp_real_robot/meshes/wheel_coupler_assembly.stl" scale = "0.001 0.001 0.001"/>  -->
             </geometry>
             <material name = 'purple'/>
